File: gartenbewaesserung.kicad_sch (KiCad schematic)
At the start: 13 parts, among them J1 24VDC IN, J2 Relais, J3 4..20mA Hydrostatischer Sensor, J4 1-Wire A, J5 1-Wire B, J6 ADS1115 Modul, Q1 IRLZ44N, U1 WeMos_D1_mini, U2 ULN2803A

Commit message: Zustand bei Fertigstellung
Parts:
- removed J4: 1-Wire A, TerminalBlock_Phoenix:TerminalBlock_Phoenix_MKDS-3-3-5.08_1x03_P5.08mm_Horizontal, symbol Connector:Screw_Terminal_01x03
- removed J5: 1-Wire B, TerminalBlock_Phoenix:TerminalBlock_Phoenix_MKDS-3-3-5.08_1x03_P5.08mm_Horizontal, symbol Connector:Screw_Terminal_01x03
- added D1: 1N5408, Diode_THT:D_DO-201AD_P15.24mm_Horizontal, symbol Diode:1N5408
- added J5: 250-206, footprints:CONN_250-206_WAG, symbol con wago 250-206:250-206
Connections:
- net +24V: now also D1.1 (K)
- net GND: now also J5.3, J5.6
- net VCC: now also J5.1, J5.4
- net at U1.12 (D3): now also J5.2, J5.5
- net at J2.1 (Pin_1): now also U2.13 (O6); no longer Q1.2 (D)
- net at J2.2 (Pin_2): now also U2.14 (O5); no longer U2.17 (O2)
- net at J2.3 (Pin_3): now also U2.15 (O4); no longer U2.16 (O3)
- net at J2.4 (Pin_4): now also U2.16 (O3); no longer U2.15 (O4)
- net at J2.5 (Pin_5): now also U2.17 (O2); no longer U2.14 (O5)
- net at J2.6 (Pin_6): now also Q1.2 (D), D1.2 (A); no longer U2.13 (O6)
- net at U1.16 (TX): no longer U2.1 (I1)
- net at U1.3 (D0): now also U2.1 (I1)
